File: KiCad/esp-iradio/esp-iradio.kicad_sch (KiCad schematic)
At the start: 0 parts

Commit message: KiCad: schematic Rev A draft, kicad-cli notes
Other:
- added sheet Audio (audio.kicad_sch)
- added sheet Controls (controls.kicad_sch)
- added sheet Display and microSD (display_sd.kicad_sch)
- added sheet Olimex socket (socket.kicad_sch)
- added sheet Power (power.kicad_sch)
Changed lines of the file:
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@@
 	(generator_version "9.0")
 	(paper "A4")
+  (sheet (at 30.0 40.0) (size 50.0 30.0) (fields_autoplaced yes)
+    (stroke (width 0.0006) (type default))
+    (fill (color 0 0 0 0.0000))
+    (property "Sheetname" "Power" (at 32.54 38.73 0)
+      (effects (font (size 1.27 1.27)) (justify left bottom))
+    )
+    (property "Sheetfile" "power.kicad_sch" (at 32.54 71.27 0)
+      (effects (font (size 1.27 1.27)) (justify left top))
+    )
+    (instances
+      (project "esp-iradio"
+        (path "/41c4da12-e59e-4675-bbd9-2603c7cfe6e6" (page "2"))
+      )
+    )
+  )
+  (sheet (at 100.0 40.0) (size 50.0 30.0) (fields_autoplaced yes)
+    (stroke (width 0.0006) (type default))
+    (fill (color 0 0 0 0.0000))
+    (property "Sheetname" "Olimex socket" (at 102.54 38.73 0)
+      (effects (font (size 1.27 1.27)) (justify left bottom))
+    )
+    (property "Sheetfile" "socket.kicad_sch" (at 102.54 71.27 0)
+      (effects (font (size 1.27 1.27)) (justify left top))
+    )
+    (instances
+      (project "esp-iradio"
+        (path "/41c4da12-e59e-4675-bbd9-2603c7cfe6e6" (page "3"))
+      )
+    )
+  )
+  (sheet (at 170.0 40.0) (size 50.0 30.0) (fields_autoplaced yes)
+    (stroke (width 0.0006) (type default))
+    (fill (color 0 0 0 0.0000))
+    (property "Sheetname" "Display and microSD" (at 172.54 38.73 0)
+      (effects (font (size 1.27 1.27)) (justify left bottom))
+    )
+    (property "Sheetfile" "display_sd.kicad_sch" (at 172.54 71.27 0)
+      (effects (font (size 1.27 1.27)) (justify left top))
+    )
+    (instances
+      (project "esp-iradio"
+        (path "/41c4da12-e59e-4675-bbd9-2603c7cfe6e6" (page "4"))
+      )
+    )
+  )
+  (sheet (at 30.0 100.0) (size 50.0 30.0) (fields_autoplaced yes)
+    (stroke (width 0.0006) (type default))
+    (fill (color 0 0 0 0.0000))
+    (property "Sheetname" "Controls" (at 32.54 98.73 0)
+      (effects (font (size 1.27 1.27)) (justify left bottom))
+    )
+    (property "Sheetfile" "controls.kicad_sch" (at 32.54 131.27 0)
+      (effects (font (size 1.27 1.27)) (justify left top))
+    )
+    (instances
+      (project "esp-iradio"
+        (path "/41c4da12-e59e-4675-bbd9-2603c7cfe6e6" (page "5"))
+      )
+    )
+  )
+  (sheet (at 100.0 100.0) (size 50.0 30.0) (fields_autoplaced yes)
+    (stroke (width 0.0006) (type default))
+    (fill (color 0 0 0 0.0000))
+    (property "Sheetname" "Audio" (at 102.54 98.73 0)
+      (effects (font (size 1.27 1.27)) (justify left bottom))
+    )
+    (property "Sheetfile" "audio.kicad_sch" (at 102.54 131.27 0)
+      (effects (font (size 1.27 1.27)) (justify left top))
+    )
+    (instances
+      (project "esp-iradio"
+        (path "/41c4da12-e59e-4675-bbd9-2603c7cfe6e6" (page "6"))
+      )
+    )
+  )
 	(sheet_instances
 		(path "/"
