File: KiCad/esp-iradio/esp-iradio.kicad_sch (KiCad schematic)
At the start: 67 parts, among them J3 LCD 1.69in ST7789 (GND VCC SC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, J4 microSD push-push, J5 Line out 3.5mm, J6 Speaker 4-8 Ohm, J7 USB-C power (GCT USB4125), J8 Spare inputs, SW1 EC11 with switch, U1 PCM5102APWR, U2 MAX98357AETE+T, U3 LM66100DCK

Commit message: KiCad: integrated board schematic Rev B (two sheets, WROVER-IE)
Co-Authored-By: Claude Opus 5.5 <noreply@anthropic.com>
Parts:
- removed C1: 10uF, Capacitor_SMD:C_0805_2012Metric, symbol Elektuur:C
- removed C2: 1uF, Capacitor_SMD:C_0603_1608Metric, symbol Elektuur:C
- removed D1: SMAJ5.0CA, Diode_SMD:D_SMA, symbol Device:D_TVS
- removed F1: 2A hold, Fuse:Fuse_1206_3216Metric, symbol Device:Polyfuse
- removed FB1: 600R@100MHz, Inductor_SMD:L_0805_2012Metric, symbol Elektuur:L
- removed FB2: 600R@100MHz 2A, Inductor_SMD:L_0805_2012Metric, symbol Elektuur:L
- removed J3: LCD 1.69in ST7789 (GND VCC SCL SDA RES DC CS BLK), Connector_PinSocket_2.54mm:PinSocket_1x08_P2.54mm_Vertical, symbol Connector_Generic:Conn_01x08
- removed J4: microSD push-push, Connector_Card:microSD_HC_Hirose_DM3AT-SF-PEJM5, symbol Connector:Micro_SD_Card
- removed J5: Line out 3.5mm, Connector_Audio:Jack_3.5mm_PJ320D_Horizontal, symbol Connector_Audio:AudioJack3
- removed J7: USB-C power (GCT USB4125), Connector_USB:USB_C_Receptacle_GCT_USB4125-xx-x_6P_TopMnt_Horizontal, symbol Connector:USB_C_Receptacle_PowerOnly_6P
- removed J8: Spare inputs, Connector_PinHeader_2.54mm:PinHeader_1x05_P2.54mm_Vertical, symbol Connector_Generic:Conn_01x05
- removed MOD1: Olimex ESP32-DevKit-LiPo, esp-iradio:Olimex_ESP32-DevKit-LiPo_Socket, symbol esp-iradio:Olimex_ESP32-DevKit-LiPo
- removed R1, R2: 5.1k 1%, Resistor_SMD:R_0603_1608Metric, symbol Elektuur:R
- removed R13, R14: 10k DNP, Resistor_SMD:R_0603_1608Metric, symbol Elektuur:R
- removed TP1: +5V_USBC, TestPoint:TestPoint_Pad_D1.5mm, symbol Connector:TestPoint
- removed TP3: GND, TestPoint:TestPoint_Pad_D1.5mm, symbol Connector:TestPoint
- removed U3: LM66100DCK, Package_TO_SOT_SMD:SOT-363_SC-70-6, symbol Power_Management:LM66100DCK
- added C25: 100nF, Capacitor_SMD:C_0603_1608Metric, symbol Elektuur:C
- added J3: LCD 1.69in ST7789V2 panel, 12-pin FPC 0.7 mm, esp-iradio:FPC_12P_P0.70mm_Solder, symbol Connector_Generic:Conn_01x12
- added J4: microSD push-push TF-01A, lcsc:TF-SMD_TF-01A, symbol esp-iradio:Micro_SD_TF01A
- added J5: Line out 3.5mm PJ-320D, lcsc:AUDIO-SMD_PJ-320D-1, symbol esp-iradio:AudioJack3_PJ320D
- added Q1: AO3400A, Package_TO_SOT_SMD:SOT-23, symbol Transistor_FET:AO3400A
- added R22: 5.6R, Resistor_SMD:R_0603_1608Metric, symbol Elektuur:R
- added R23: 100k, Resistor_SMD:R_0603_1608Metric, symbol Elektuur:R
- added U3: ESP32-WROVER-IE-N16R8, lcsc:ESP32-WROVER-IE_SMD, symbol esp-iradio:ESP32-WROVER-IE_iRadio
- TP2: value +VAMP -> VSYS
Connections:
- net +3V3: now also R21.2 (-), C25.1 (+), J3.3 (Pin_3), J3.4 (Pin_4), J4.4 (VDD), U3.2 (3V3)
- net GND: now also C25.2 (-), J3.1 (Pin_1), J3.12 (Pin_12), J3.5 (Pin_5), J3.6 (Pin_6), J4.10 (SHIELD), J4.11 (SHIELD), J4.12 (SHIELD), J4.13 (SHIELD), J4.6 (VSS), J5.1 (S), Q1.2 (S), R23.1 (+), U3.1 (GND), U3.15 (GND), U3.38 (GND), U3.39 (GND)
- net at TP6.1, U1.13 (BCK), U2.16 (BCLK): now also U3.12 (IO27)
- net at TP7.1, U1.15 (LRCK), U2.14 (LRCLK): now also U3.13 (IO14)
- net at TP8.1, U1.14 (DIN), U2.1 (DIN): now also U3.16 (IO13)
- net at R9.1 (+): now also U3.37 (IO23)
- net at R5.1 (+): now also J4.7 (DAT0), U3.31 (IO19)
- net at R8.1 (+), TP5.1: now also U3.30 (IO18)
- net at R3.1 (+): now also J3.8 (Pin_8), U3.29 (IO5)
- net at R4.2 (-): now also J4.2 (DAT3/CD), U3.26 (IO4)
- net at R21.1 (+), U2.4 (~{SD_MODE}): now also U3.24 (IO2)
- net at C6.1 (+), R10.2 (-), SW1.A: now also U3.8 (IO32)
- net at C7.1 (+), R11.2 (-), SW1.B: now also U3.9 (IO33)
- net at C8.1 (+), R12.2 (-), SW1.S1: now also U3.10 (IO25)
- net at C18.1 (+), R16.2 (-): now also J5.4 (T)
- net at R9.2 (-): now also J3.10 (Pin_10), J4.3 (CMD)
- net at R6.1 (+): now also J4.8 (DAT1)
- net at R8.2 (-): now also J3.9 (Pin_9), J4.5 (CLK)
- net at R7.2 (-): now also J4.1 (DAT2)
- net at C19.1 (+), R17.2 (-): now also J5.2 (R)
- net +VAMP renamed VSYS
- net VSYS: no longer R21.2 (-)
- new net: J3.11 (Pin_11), U3.33 (IO21)
- new net: J3.2 (Pin_2), R22.2 (-)
- new net: J3.7 (Pin_7), U3.36 (IO22)
- new net: Q1.1 (G), R23.2 (-), U3.11 (IO26)
- new net: Q1.3 (D), R22.1 (+)
- new net CHG: U3.6 (IO34)
- new net ESP_EN: U3.3 (EN)
- new net ESP_IO0: U3.25 (IO0)
- new net PGOOD: U3.4 (IO36)
- new net RXD0: U3.34 (RXD0)
- new net TXD0: U3.35 (TXD0)
- new net VBAT_SENSE: U3.7 (IO35)
- new net VBUS_SENSE: U3.5 (IO39)
- no-connect marks 19 -> 3
Other:
- added sheet Power, charger and USB (power_usb.kicad_sch)
- note added: "AUDIO: PCM5102A DAC, 3.5 mm line out, MAX98357A I2S mono amplifier (VSYS)"
- note added: "CONTROLS: EC11 encoder (recessed knob)"
- note added: "Sheet 2: USB-C, CH340C, BQ24074 charger,"
- note added: "cell protection, 3.3 V LDO, +3V3A for the DAC"
- note removed: "AUDIO: PCM5102A DAC, 3.5 mm line out, MAX98357A I2S mono amplifier"
- note removed: "CONTROLS: EC11 encoder, spare inputs"
- note removed: "POWER: USB-C 5 V in, ideal diode to the Olimex 5 V pin"
- title: ESP iRadio carrier board -> ESP iRadio integrated board - radio

Commit message: KiCad Rev B: review changes agreed with Grok
Co-Authored-By: Claude Opus 5.5 <noreply@anthropic.com>
Parts:
- removed C24: 220uF 10V, Capacitor_SMD:CP_Elec_6.3x7.7, symbol Elektuur:C-polar
- J6: LCSC (none) -> C131337
- U1: LCSC (none) -> C107671
- U2: footprint Package_DFN_QFN:TQFN-16-1EP_3x3mm_P0.5mm_EP1.23x1.23mm -> Package_DFN_QFN:TQFN-16-1EP_3x3mm_P0.5mm_EP1.23x1.23mm_ThermalVias; LCSC (none) -> C910544
Changed lines of the file:
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@@
 			)
 		)
+		(property "LCSC" "C107671"
+			(at 200.66 218.44 0)
+			(effects
+				(font
+					(size 1.27 1.27)
+				)
+				(hide yes)
+			)
+		)
 		(pin "15"
 		)
@@
 			)
 		)
-		(property "Footprint" "Package_DFN_QFN:TQFN-16-1EP_3x3mm_P0.5mm_EP1.23x1.23mm"
+		(property "Footprint" "Package_DFN_QFN:TQFN-16-1EP_3x3mm_P0.5mm_EP1.23x1.23mm_ThermalVias"
 			(at 320.04 175.26 0)
 			(effects
@@
 			)
 		)
+		(property "LCSC" "C910544"
+			(at 320.04 175.26 0)
+			(effects
+				(font
+					(size 1.27 1.27)
+				)
+				(hide yes)
+			)
+		)
 		(pin "1"
 		)
@@
 			)
 		)
+		(property "LCSC" "C131337"
+			(at 345.44 167.64 0)
+			(effects
+				(font
+					(size 1.27 1.27)
+				)
+				(hide yes)
+			)
+		)
 		(pin "1"
 		)
@@
 	)
 	(symbol
-		(lib_id "Elektuur:C-polar")
-		(at 370.84 210.82 0)
-		(unit 1)
-		(exclude_from_sim no)
-		(in_bom yes)
-		(on_board yes)
-		(dnp no)
-		(property "Reference" "C24"
-			(at 374.65 209.55 0)
-			(effects
-				(font
-					(size 1.27 1.27)
-				)
-				(justify left)
-			)
-		)
-		(property "Value" "220uF 10V"
-			(at 374.65 212.09 0)
-			(effects
-				(font
-					(size 1.27 1.27)
-				)
-				(justify left)
-			)
-		)
-		(property "Footprint" "Capacitor_SMD:CP_Elec_6.3x7.7"
-			(at 370.84 210.82 0)
-			(effects
-				(font
-					(size 1.27 1.27)
-				)
-				(hide yes)
-			)
-		)
-		(property "Datasheet" ""
-			(at 370.84 210.82 0)
-			(effects
-				(font
-					(size 1.27 1.27)
-				)
-				(hide yes)
-			)
-		)
-		(pin "1"
-		)
-		(pin "2"
-		)
-		(instances
-			(project "esp-iradio"
-				(path "/41c4da12-e59e-4675-bbd9-2603c7cfe6e6"
-					(reference "C24")
-					(unit 1)
-				)
-			)
-		)
-	)
-	(symbol
-		(lib_id "Elektuur:V-+")
-		(at 370.84 205.74 180)
-		(unit 1)
-		(exclude_from_sim no)
-		(in_bom yes)
-		(on_board yes)
-		(dnp no)
-		(property "Reference" "#PWR066"
-			(at 370.84 205.74 0)
-			(effects
-				(font
-					(size 1.27 1.27)
-				)
-				(hide yes)
-			)
-		)
-		(property "Value" "VSYS"
-			(at 370.84 199.39 0)
-			(effects
-				(font
-					(size 1.27 1.27)
-				)
-				(hide yes)
-			)
-		)
-		(property "Footprint" ""
-			(at 370.84 205.74 0)
-			(effects
-				(font
-					(size 1.27 1.27)
-				)
-				(hide yes)
-			)
-		)
-		(property "Datasheet" ""
-			(at 370.84 205.74 0)
-			(effects
-				(font
-					(size 1.27 1.27)
-				)
-				(hide yes)
-			)
-		)
-		(pin "0"
-		)
-		(instances
-			(project "esp-iradio"
-				(path "/41c4da12-e59e-4675-bbd9-2603c7cfe6e6"
-					(reference "#PWR066")
-					(unit 1)
-				)
-			)
-		)
-	)
-	(symbol
-		(lib_id "Elektuur:V-GND")
-		(at 370.84 215.9 0)
-		(unit 1)
-		(exclude_from_sim no)
-		(in_bom yes)
-		(on_board yes)
-		(dnp no)
-		(property "Reference" "#PWR067"
-			(at 370.84 215.9 0)
-			(effects
-				(font
-					(size 1.27 1.27)
-				)
-				(hide yes)
-			)
-		)
-		(property "Value" "GND"
-			(at 370.84 215.9 0)
-			(effects
-				(font
-					(size 1.27 1.27)
-				)
-				(hide yes)
-			)
-		)
-		(property "Footprint" ""
-			(at 370.84 215.9 0)
-			(effects
-				(font
-					(size 1.27 1.27)
-				)
-				(hide yes)
-			)
-		)
-		(property "Datasheet" ""
-			(at 370.84 215.9 0)
-			(effects
-				(font
-					(size 1.27 1.27)
-				)
-				(hide yes)
-			)
-		)
-		(pin "0"
-		)
-		(instances
-			(project "esp-iradio"
-				(path "/41c4da12-e59e-4675-bbd9-2603c7cfe6e6"
-					(reference "#PWR067")
-					(unit 1)
-				)
-			)
-		)
-	)
-	(symbol
 		(lib_id "Connector:TestPoint")
 		(at 391.16 205.74 0)
@@
 		(on_board yes)
 		(dnp no)
-		(property "Reference" "#PWR068"
+		(property "Reference" "#PWR066"
 			(at 391.16 205.74 0)
 			(effects
@@
 			(project "esp-iradio"
 				(path "/41c4da12-e59e-4675-bbd9-2603c7cfe6e6"
-					(reference "#PWR068")
+					(reference "#PWR066")
 					(unit 1)
 				)
@@
 		(on_board yes)
 		(dnp no)
-		(property "Reference" "#PWR069"
+		(property "Reference" "#PWR067"
 			(at 391.16 50.8 0)
 			(effects
@@
 			(project "esp-iradio"
 				(path "/41c4da12-e59e-4675-bbd9-2603c7cfe6e6"
-					(reference "#PWR069")
+					(reference "#PWR067")
 					(unit 1)
 				)

Commit message: KiCad Rev B: first layout (80 x 60 mm, 4 layers, autorouted)
Co-Authored-By: Claude Opus 5.5 <noreply@anthropic.com>
Parts:
- H1, H2, H3, H4, J3, TP2, TP4, TP5, TP6, TP7, TP8: now left out of the parts list
Changed lines of the file:
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@@
 		(unit 1)
 		(exclude_from_sim no)
-		(in_bom yes)
+		(in_bom no)
 		(on_board yes)
 		(dnp no)
@@
 		(unit 1)
 		(exclude_from_sim no)
-		(in_bom yes)
+		(in_bom no)
 		(on_board yes)
 		(dnp no)
@@
 		(unit 1)
 		(exclude_from_sim no)
-		(in_bom yes)
+		(in_bom no)
 		(on_board yes)
 		(dnp no)
@@
 		(unit 1)
 		(exclude_from_sim no)
-		(in_bom yes)
+		(in_bom no)
 		(on_board yes)
 		(dnp no)
@@
 		(unit 1)
 		(exclude_from_sim no)
-		(in_bom yes)
+		(in_bom no)
 		(on_board yes)
 		(dnp no)
@@
 		(unit 1)
 		(exclude_from_sim no)
-		(in_bom yes)
+		(in_bom no)
 		(on_board yes)
 		(dnp no)
@@
 		(unit 1)
 		(exclude_from_sim no)
-		(in_bom yes)
+		(in_bom no)
 		(on_board yes)
 		(dnp no)
@@
 		(unit 1)
 		(exclude_from_sim no)
-		(in_bom yes)
+		(in_bom no)
 		(on_board yes)
 		(dnp no)
@@
 		(unit 1)
 		(exclude_from_sim no)
-		(in_bom yes)
+		(in_bom no)
 		(on_board yes)
 		(dnp no)
@@
 		(unit 1)
 		(exclude_from_sim no)
-		(in_bom yes)
+		(in_bom no)
 		(on_board yes)
 		(dnp no)
@@
 		(unit 1)
 		(exclude_from_sim no)
-		(in_bom yes)
+		(in_bom no)
 		(on_board yes)
 		(dnp no)

Commit message: KiCad Rev B: HS20S010B display module on sockets, 90 x 60 mm board
Co-Authored-By: Claude Opus 5.5 <noreply@anthropic.com>
Parts:
- removed Q1: AO3400A, Package_TO_SOT_SMD:SOT-23, symbol Transistor_FET:AO3400A
- removed R22: 5.6R, Resistor_SMD:R_0603_1608Metric, symbol Elektuur:R
- removed R23: 100k, Resistor_SMD:R_0603_1608Metric, symbol Elektuur:R
- added H5, H6, H7: M2.5, MountingHole:MountingHole_2.7mm_M2.5, symbol Mechanical:MountingHole
- added J7: Display CN2 (mechanical), Connector_PinSocket_2.54mm:PinSocket_1x10_P2.54mm_Vertical, symbol Connector_Generic:Conn_01x10
- H1: value M3 -> M2.5; footprint MountingHole:MountingHole_3.2mm_M3 -> MountingHole:MountingHole_2.7mm_M2.5
- J3: value LCD 1.69in ST7789V2 panel, 12-pin FPC 0.7 mm -> Display HS20S010B CN1; footprint esp-iradio:FPC_12P_P0.70mm_Solder -> Connector_PinSocket_2.54mm:PinSocket_1x10_P2.54mm_Vertical; symbol Connector_Generic:Conn_01x12 -> Connector_Generic:Conn_01x10; LCSC (none) -> C2897373; now in the parts list
Connections:
- net +3V3: now also J3.2 (Pin_2); no longer J3.3 (Pin_3), J3.4 (Pin_4)
- net GND: no longer J3.12 (Pin_12), J3.5 (Pin_5), J3.6 (Pin_6)
- net LCD_BL: now reaches U3.11 (IO26)
- net LCD_BL: now also J3.8 (Pin_8)
- net at R3.1 (+), U3.29 (IO5): now also J3.7 (Pin_7); no longer J3.8 (Pin_8)
- net at U3.33 (IO21): now also J3.5 (Pin_5); no longer J3.11 (Pin_11)
- net at U3.36 (IO22): now also J3.6 (Pin_6); no longer J3.7 (Pin_7)
- net at J4.5 (CLK), R8.2 (-): now also J3.3 (Pin_3); no longer J3.9 (Pin_9)
- net at J4.3 (CMD), R9.2 (-): now also J3.4 (Pin_4); no longer J3.10 (Pin_10)
- no-connect marks 3 -> 15
Other:
- note added: "DISPLAY MODULE (2.0in ST7789, SPI) AND microSD"
- note added: "Module LCSC C5329586 (loose part)"
- note removed: "DISPLAY (ST7789, SPI) AND microSD"
- moved on the sheet: C25, C5

Commit message: KiCad Rev C: hand assembly (1206), RCA outputs, display/encoder/connectors floor plan
Co-Authored-By: Claude Opus 5.5 <noreply@anthropic.com>
Parts:
- added H8: M3, MountingHole:MountingHole_3.2mm_M3, symbol Mechanical:MountingHole
- added J8: Line out RCA L/R AV-210-WR, lcsc:RCA-TH_AV-210-WR, symbol Connector_Generic:Conn_01x04
- C10, C12, C14, C22, C3, C5: footprint Capacitor_SMD:C_0805_2012Metric -> Capacitor_SMD:C_1206_3216Metric
- C11, C13, C15, C16, C17, C18, C19, C23, C25, C4, C6, C7, C8, C9: footprint Capacitor_SMD:C_0603_1608Metric -> Capacitor_SMD:C_1206_3216Metric
- R10, R11, R12, R15, R16, R17, R21, R3, R4, R5, R6, R7, R8, R9: footprint Resistor_SMD:R_0603_1608Metric -> Resistor_SMD:R_1206_3216Metric
Connections:
- net GND: now also J8.1 (Pin_1), J8.3 (Pin_3)
- net at C19.1 (+), J5.2 (R), R17.2 (-): now also J8.4 (Pin_4)
- net at C18.1 (+), J5.4 (T), R16.2 (-): now also J8.2 (Pin_2)
