File: KiCad/esp-iradio/esp-iradio.kicad_sch (KiCad schematic)
At the start: 58 parts, among them J3 Display HS20S010B CN1, J4 microSD push-push TF-01A, J5 Line out 3.5mm PJ-320D, J6 Speaker 4-8 Ohm, J7 Display CN2 (mechanical), J8 Line out RCA L/R AV-210-WR, SW1 EC11 with switch, U1 PCM5102APWR, U2 MAX98357AETE+T, U3 ESP32-WROVER-IE-N16R8

Commit message: 3D models for the USB-C and the encoder (project footprints, EasyEDA models)
Co-Authored-By: Claude Opus 5.5 <noreply@anthropic.com>
Parts:
- SW1: footprint Rotary_Encoder:RotaryEncoder_Alps_EC11E-Switch_Vertical_H20mm -> esp-iradio:RotaryEncoder_Alps_EC11E-Switch_Vertical_H20mm
Changed lines of the file:
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@@
 			)
 		)
-		(property "Footprint" "Rotary_Encoder:RotaryEncoder_Alps_EC11E-Switch_Vertical_H20mm"
+		(property "Footprint" "esp-iradio:RotaryEncoder_Alps_EC11E-Switch_Vertical_H20mm"
 			(at 40.64 129.54 0)
 			(effects

Commit message: 3D: display module on J3, solid PJ-320D model
Co-Authored-By: Claude Opus 5.5 <noreply@anthropic.com>
Parts:
- J3: footprint Connector_PinSocket_2.54mm:PinSocket_1x10_P2.54mm_Vertical -> esp-iradio:PinSocket_1x10_P2.54mm_Vertical_HS20S010B
Changed lines of the file:
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@@
 			)
 		)
-		(property "Footprint" "Connector_PinSocket_2.54mm:PinSocket_1x10_P2.54mm_Vertical"
+		(property "Footprint" "esp-iradio:PinSocket_1x10_P2.54mm_Vertical_HS20S010B"
 			(at 345.44 63.5 0)
 			(effects
