File: KiCad/esp-iradio/esp-iradio.kicad_sch (KiCad schematic)
At the start: 58 parts, among them J3 Display HS20S010B CN1, J4 microSD push-push TF-01A, J5 Line out 3.5mm PJ-320D, J6 Speaker 4-8 Ohm, J7 Display CN2 (mechanical), J8 Line out RCA L/R AV-210-WR, SW1 EC11 with switch, U1 PCM5102APWR, U2 MAX98357AETE+T, U3 ESP32-WROVER-IE-N16R8

Commit message: Speaker J6 as a 5.0 mm screw terminal; switch and encoder 3D models on their holes
Parts:
- J6: footprint Connector_JST:JST_PH_B2B-PH-K_1x02_P2.00mm_Vertical -> esp-iradio:TerminalBlock_MaiXu_MX126-5.0-02P_1x02_P5.00mm; LCSC C131337 -> C8404
Changed lines of the file:
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@@
 			)
 		)
-		(property "Footprint" "Connector_JST:JST_PH_B2B-PH-K_1x02_P2.00mm_Vertical"
+		(property "Footprint" "esp-iradio:TerminalBlock_MaiXu_MX126-5.0-02P_1x02_P5.00mm"
 			(at 345.44 167.64 0)
 			(effects
@@
 			)
 		)
-		(property "LCSC" "C131337"
+		(property "LCSC" "C8404"
 			(at 345.44 167.64 0)
 			(effects
