File: KiCad/esp-iradio/esp-iradio.kicad_pcb (KiCad board)
At the start: 4 copper layers, 122 x 76 mm, 122 parts, among them J201 USB-C TYPE-C-31-M-12, J202 Li-Po cell (JST-PH), J3 Display HS20S010B CN1, J4 microSD push-push TF-01A, J5 Line out 3.5mm PJ-320D, J6 Speaker 4-8 Ohm, J7 Display CN2 (mechanical), J8 Line out RCA L/R AV-210-WR, Q201 MMBT3904, Q202 MMBT3904, Q203 DMG2305UX-7, SW1 EC11 with switch, SW201 RESET, SW202 BOOT, SW203 ON/OFF MSK12C02, U1 PCM5102APWR, U2 MAX98357AETE+T, U201 BQ24074RGTT, U202 USBLC6-2SC6, U203 CH340C, U204 DW01A, U205 FS8205A, U206 AP7361C-33Y5-13, U207 TPLP5907MFX-3.3, U3 ESP32-WROVER-IE-N16R8

Commit message: USB-C 0.5 mm past the bottom edge
Parts:
- moved J201 0.50 mm to (177.0, 172.8)
Routing:
- net /Power, charger and USB/EN_3V3: track 127.1 -> 108.4 mm
- net Net-(U204-OD): track 7.25 -> 20.1 mm
- net /Power, charger and USB/VIN: track 89.1 -> 100.7 mm
- net Net-(R17-+): track 25.8 -> 14.4 mm, vias 0 -> 2
- net Net-(R21-+): track 86.9 -> 97.9 mm, vias 2 -> 3
- net ESP_EN: track 122.7 -> 133.2 mm, vias 3 -> 2
- net ESP_IO0: track 137.3 -> 146.7 mm, vias 3 -> 5
- net Net-(U204-OC): track 9.81 -> 18.3 mm
- net Net-(R210-+): track 22.4 -> 14.1 mm, vias 0 -> 2
- net +3V3: track 324.2 -> 332.0 mm, vias 1 -> 4
- net Net-(J3-Pin_4): track 119.9 -> 112.5 mm
- net /Power, charger and USB/BATN: track 35.0 -> 28.7 mm, vias 0 -> 1
- net /Power, charger and USB/USB_D+: track 21.3 -> 15.1 mm, vias 0 -> 2
- net Net-(C8-+): track 56.5 -> 50.6 mm, vias 1 -> 2
- net /Power, charger and USB/USB_D-: track 17.5 -> 11.6 mm
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
Commit message: Board centred in the A4 drawing frame (origin in placement.py)
Parts:
- moved C15 35.3 mm to (100.0, 113.8)
- moved C16 35.3 mm to (96.0, 113.8)
- moved C17 35.3 mm to (113.0, 113.8)
- moved C18 35.3 mm to (101.8, 125.8)
- moved C19 35.3 mm to (114.4, 125.8)
- moved C205 35.3 mm to (190.5, 114.3)
- moved C208 35.3 mm to (104.5, 98.8)
- moved C209 35.3 mm to (108.5, 98.8)
- moved C7 35.3 mm to (133.0, 113.8)
- moved D201 35.3 mm to (169.0, 120.3)
- moved Q202 35.3 mm to (181.5, 114.3)
- moved R11 35.3 mm to (137.0, 113.8)
- moved R15 35.3 mm to (117.0, 113.8)
- moved R16 35.3 mm to (95.5, 125.8)
- moved R17 35.3 mm to (108.1, 125.8)
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Routing:
- net ESP_IO0: track 146.7 -> 174.8 mm, vias 5 -> 3
- net /Power, charger and USB/VIN: track 100.7 -> 87.6 mm
- net Net-(R17-+): track 14.4 -> 25.8 mm, vias 2 -> 0
- net Net-(C8-+): track 50.6 -> 61.7 mm
- net Net-(U204-OC): track 18.3 -> 7.61 mm
- net Net-(U204-OD): track 20.1 -> 9.90 mm
- net +3V3: track 332.0 -> 321.9 mm, vias 4 -> 1
- net Net-(Q202-E): track 19.5 -> 29.3 mm
- net ESP_EN: track 133.2 -> 124.1 mm
- net Net-(R21-+): track 97.9 -> 89.2 mm, vias 3 -> 4
- net Net-(C7-+): track 33.1 -> 40.3 mm, vias 1 -> 2
- net VSYS: track 219.9 -> 226.2 mm, vias 5 -> 4
- net CHG: track 85.9 -> 92.1 mm, vias 2 -> 0
- net /Power, charger and USB/USB_D-: track 11.6 -> 17.6 mm, vias 2 -> 0
- net Net-(R220-+): track 12.8 -> 18.1 mm, vias 2 -> 0
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
Commit message: Speaker J6 as a 5.0 mm screw terminal; switch and encoder 3D models on their holes
Parts:
- J6: footprint Connector_JST:JST_PH_B2B-PH-K_1x02_P2.00mm_Vertical -> esp-iradio:TerminalBlock_MaiXu_MX126-5.0-02P_1x02_P5.00mm
- moved J6 5.63 mm to (179.5, 138.0), turned to 180 degrees
- moved SW203 4.50 mm to (188.0, 139.6)
Routing:
- net ESP_IO0: track 174.8 -> 150.3 mm
- net Net-(R21-+): track 89.2 -> 106.8 mm
- net Net-(J3-Pin_3): track 98.4 -> 113.4 mm
- net Net-(R17-+): track 25.8 -> 12.6 mm
- net Net-(Q202-E): track 29.3 -> 19.6 mm
- net VSYS: track 226.2 -> 216.7 mm
- net TXD0: track 97.7 -> 107.0 mm
- net /Power, charger and USB/USB_D+: track 20.2 -> 11.7 mm
- net +3V3: track 321.9 -> 313.8 mm, vias 1 -> 3
- net CHG: track 92.1 -> 84.3 mm, vias 0 -> 2
- net /Power, charger and USB/USB_D-: track 17.6 -> 10.0 mm
- net Net-(J202-Pin_1): track 33.5 -> 41.0 mm, vias 0 -> 1
- net VBUS_SENSE: track 78.1 -> 85.4 mm
- net Net-(U1-BCK): track 124.0 -> 130.3 mm, vias 3 -> 4
- net /Power, charger and USB/CHG_N: track 67.2 -> 73.4 mm
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
Commit message: Edge connectors spread over the width; screw terminal openings at the edge
Parts:
- moved SW203 7.65 mm to (195.7, 139.6)
- moved J201 4.75 mm to (169.2, 139.8)
- moved U202 4.75 mm to (166.8, 129.0)
- moved J4 4.35 mm to (152.8, 133.4)
- moved C3 3.70 mm to (141.7, 131.5)
- moved C4 3.70 mm to (141.7, 138.0)
- moved J5 2.85 mm to (132.8, 133.5)
- moved J8 2.05 mm to (113.2, 134.8)
- moved J6 1.70 mm to (180.7, 139.2), turned to 0 degrees
- moved D202 0.85 mm to (192.4, 133.0)
- moved D203 0.72 mm to (198.2, 133.0)
Routing:
- net +3V3: track 313.8 -> 343.4 mm, vias 3 -> 1
- net Net-(J4-DAT3/CD): track 59.9 -> 88.7 mm
- net Net-(J3-Pin_3): track 113.4 -> 94.5 mm
- net /Power, charger and USB/VBUS: track 18.3 -> 35.0 mm
- net VSYS: track 216.7 -> 230.1 mm, vias 4 -> 5
- net Net-(R17-+): track 12.6 -> 25.8 mm
- net TXD0: track 107.0 -> 94.0 mm
- net Net-(J6-Pin_2): track 27.3 -> 15.1 mm
- net RXD0: track 97.1 -> 87.4 mm
- net /Power, charger and USB/EN_3V3: track 116.5 -> 126.1 mm
- net /Power, charger and USB/VBAT: track 51.9 -> 42.5 mm, vias 2 -> 3
- net Net-(J3-Pin_4): track 113.6 -> 104.5 mm
- net /Power, charger and USB/CHG_N: track 73.4 -> 64.7 mm
- net Net-(R210-+): track 22.4 -> 14.9 mm, vias 0 -> 2
- net +3V3A: track 48.4 -> 55.4 mm, vias 2 -> 0
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
Commit message: Keep-out under the USB-C shell: no vias or F.Cu tracks (Grok round 10)
Routing:
- net Net-(J3-Pin_3): track 94.5 -> 121.3 mm
- net Net-(J3-Pin_4): track 104.5 -> 126.4 mm, vias 2 -> 3
- net +3V3: track 343.4 -> 325.9 mm
- net Net-(J4-DAT3/CD): track 88.7 -> 75.6 mm, vias 3 -> 4
- net /Power, charger and USB/EN_3V3: track 126.1 -> 138.2 mm, vias 4 -> 3
- net /Power, charger and USB/USB_D+: track 12.4 -> 24.5 mm, vias 0 -> 2
- net Net-(R21-+): track 104.1 -> 92.2 mm, vias 2 -> 3
- net VBUS_SENSE: track 87.1 -> 76.1 mm
- net Net-(R210-+): track 14.9 -> 22.4 mm, vias 2 -> 0
- net VSYS: track 230.1 -> 222.7 mm, vias 5 -> 6
- net /Power, charger and USB/USB_D-: track 13.7 -> 21.0 mm, vias 2 -> 0
- net +3V3A: track 55.4 -> 48.5 mm
- net Net-(J4-DAT0): track 67.8 -> 61.4 mm
- net Net-(J201-CC2): track 13.8 -> 7.58 mm, vias 2 -> 0
- net /Power, charger and USB/PGOOD_N: track 69.6 -> 63.7 mm, vias 2 -> 3
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